Commit message: prepared kr210 r3100 robot

File: kuka_quantec_support/urdf/kr210_r3100_2.urdf (robot description, URDF)
Before this commit: robot kr210_r2700_2, 11 links, 10 joints
Links:
- link base_link: geometry collision mesh filename=package://kuka_quantec_support/meshes/kr210_r3100_2/collisi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; visual mesh filename=package://kuka_quantec_support/meshes/kr210_r3100_2/visual/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
- link link_1: geometry collision mesh filename=package://kuka_quantec_support/meshes/kr210_r3100_2/collisi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; visual mesh filename=package://kuka_quantec_support/meshes/kr210_r3100_2/visual/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
- link link_2: geometry collision mesh filename=package://kuka_quantec_support/meshes/kr210_r3100_2/collisi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; visual mesh filename=package://kuka_quantec_support/meshes/kr210_r3100_2/visual/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
- link link_3: geometry collision mesh filename=package://kuka_quantec_support/meshes/kr210_r3100_2/collisi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; visual mesh filename=package://kuka_quantec_support/meshes/kr210_r3100_2/visual/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
- link link_4: geometry collision mesh filename=package://kuka_quantec_support/meshes/kr210_r3100_2/collisi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; visual mesh filename=package://kuka_quantec_support/meshes/kr210_r3100_2/visual/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
- link link_5: geometry collision mesh filename=package://kuka_quantec_support/meshes/kr210_r3100_2/collisi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; visual mesh filename=package://kuka_quantec_support/meshes/kr210_r3100_2/visual/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
- link link_6: geometry collision mesh filename=package://kuka_quantec_support/meshes/kr210_r3100_2/collisi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; visual mesh filename=package://kuka_quantec_support/meshes/kr210_r3100_2/visual/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
Joints:
- joint joint_1: limit lower=-3.2288591161895095E0 upper=3.2288591161895095E0 effort=7290 velocity=2.0384 -> lower=-3.2288591161895095E0 upper=3.2288591161895095E0 effort=7290 velocity=1.8326
- joint joint_2: limit lower=-2.443460952792061E0 upper=-8.726646259971647E-2 effort=8910 velocity=1.9451 -> lower=-2.443460952792061E0 upper=-8.726646259971647E-2 effort=8910 velocity=1.64061
- joint joint_3: limit lower=-2.0943951023931953E0 upper=2.9321531433504737E0 effort=6988.84717 velocity=1.95477 -> lower=-2.0943951023931953E0 upper=2.9321531433504737E0 effort=7251.2876 velocity=1.74533; origin xyz=1.15 0.0 0.0 rpy=0.0 0.0 -1.5707963267948963 -> xyz=1.35 0.0 0.0 rpy=0.0 0.0 -1.5707963267948963
- joint joint_4: limit lower=-6.1086523819801535E0 upper=6.1086523819801535E0 effort=2274.29199 velocity=3.12414 -> lower=-6.1086523819801535E0 upper=6.1086523819801535E0 effort=2356.12598 velocity=2.37365
- joint joint_5: limit lower=-2.181661564992912E0 upper=2.181661564992912E0 effort=1398.30298 velocity=3.00197 -> lower=-2.138028333693054E0 upper=2.138028333693054E0 effort=2358.44531 velocity=2.25147; origin xyz=0.0 0.0 -1.22 rpy=-1.5707963267948963 0.0 -0.0 -> xyz=0.0 0.0 -1.42 rpy=-1.5707963267948963 0.0 -0.0
- joint joint_6: limit lower=-6.1086523819801535E0 upper=6.1086523819801535E0 effort=781.554626 velocity=3.83972 -> lower=-6.1086523819801535E0 upper=6.1086523819801535E0 effort=1508.75476 velocity=3.59538
- joint link6-flange: origin xyz=0.0 0.0 -0.215 rpy=0 1.57079632679 -0.0 -> xyz=0.0 0.0 -0.240 rpy=0 1.57079632679 -0.0
- joint link6-tool0: origin xyz=0.0 0.0 -0.215 rpy=0 3.14159265359 -0.0 -> xyz=0.0 0.0 -0.240 rpy=0 3.14159265359 -0.0
